File: EthernetDesignBlocks.kicad_blocks/LAN8650.kicad_block/LAN8650.kicad_pcb (KiCad board)
At the start: 2 copper layers, 36 parts, among them U2 LAN8650B1-E/LMX, U3 LP38852MRX-ADJ/NOPB

Commit message: UPDATED
Parts:
- removed C1: 100n, Capacitor_SMD:C_0402_1005Metric
- removed C10, C11, C12, C9: 10u, Capacitor_SMD:C_0402_1005Metric
- removed C13, C15, C17, C19, C21: 10n, Capacitor_SMD:C_0402_1005Metric
- removed C14, C16, C18, C20, C22, C23, C24, C25: .1U, Capacitor_SMD:C_0402_1005Metric
- removed C2, C3, C4, C5, C6, C7, C8: 1u, Capacitor_SMD:C_0402_1005Metric
- removed R1: 2.94K, Resistor_SMD:R_0402_1005Metric
- removed R2: 1.13K, Resistor_SMD:R_0402_1005Metric
- removed R3: 12.4K, Resistor_SMD:R_0402_1005Metric
- removed R4, R5: 10K, Resistor_SMD:R_0402_1005Metric
- removed R6, R7: 49.9K, Resistor_SMD:R_0402_1005Metric
- removed R8: 100K, Resistor_SMD:R_0402_1005Metric
- removed U2: LAN8650B1-E/LMX, Package_DFN_QFN:QFN-32-1EP_5x5mm_P0.5mm_EP3.1x3.1mm
- removed U3: LP38852MRX-ADJ/NOPB, Package_SO:SOIC-8-1EP_3.9x4.9mm_P1.27mm_EP2.29x3mm_ThermalVias
- removed XTAL1: ECS-2520S33-250-FN-TR, GaladyneOscillatorFootprintsLibrary:ECS-2520S_ECS
Routing:
- net (no net): track 0.00 -> 27.8 mm
- net /Ethernet/ETH_10T1S_TRXN_N: track 8.59 -> 0.00 mm
- net /Ethernet/TRXN_N: track 7.15 -> 0.00 mm
- net /Ethernet/TRXP_P: track 5.43 -> 0.00 mm
- net /Ethernet/ETH_10T1S_TRXP_P: track 4.87 -> 0.00 mm
- net Net-(C25-Pad2): track 3.41 -> 0.00 mm
- net GND: track 34.8 -> 32.6 mm, vias 12 -> 10
- net +3V3: track 37.6 -> 39.8 mm, vias 3 -> 5
- net Net-(C23-Pad2): track 0.00 -> 1.68 mm
